File: memboard.kicad_pcb (KiCad board)
At the start: 4 copper layers, 23 x 51 mm, 40 parts, among them J1 USB_C_Receptacle_USB2.0_14P, J2 Conn_01x20_Pin, J3 Conn_01x20_Pin, J4 Conn_01x03_Socket, SW1 SW_Push, SW2 SW_Push, U3 RP2354A, U4 APS6404L-3SQRx-ZR, U5 AP2112K-3.3, Y1 12 MHz

Commit message: Added a Schottky diode to allow power through VBUS because USB-C cannot be back powered
Parts:
- added D1: PMEG2010BER, Diode_SMD:Nexperia_CFP3_SOD-123W, B.Cu at (140.4, 40.5)
Connections:
- J1 pad A4: VBUS -> Net-(D1-A)
- J1 pad A9: VBUS -> Net-(D1-A)
- J1 pad B4: VBUS -> Net-(D1-A)
- J1 pad B9: VBUS -> Net-(D1-A)
Routing:
- net Net-(D1-A): track 0.00 -> 10.7 mm, vias 0 -> 1
- net VBUS: track 24.1 -> 26.7 mm, vias 0 -> 1
- added copper zone on In1.Cu, net GND
- added copper zone on In2.Cu, net GND
