File: memboard.kicad_sch (KiCad schematic)
At the start: 40 parts, among them J1 USB_C_Receptacle_USB2.0_14P, J2 Conn_01x20_Pin, J3 Conn_01x20_Pin, J4 Conn_01x03_Socket, SW1 SW_Push, SW2 SW_Push, U3 RP2354A, U4 APS6404L-3SQRx-ZR, U5 AP2112K-3.3, Y1 12 MHz

Commit message: Added a Schottky diode to allow power through VBUS because USB-C cannot be back powered
Parts:
- added D1: PMEG2010BER, Diode_SMD:Nexperia_CFP3_SOD-123W, symbol Diode:PMEG2010BER
Connections:
- net VBUS: now also D1.1 (K); no longer J1.A4 (VBUS), J1.A9 (VBUS), J1.B4 (VBUS), J1.B9 (VBUS)
- new net: D1.2 (A), J1.A4 (VBUS), J1.A9 (VBUS), J1.B4 (VBUS), J1.B9 (VBUS)
Changed lines of the file:
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@@
 	)
 	(junction
-		(at 77.47 29.21)
-		(diameter 0)
-		(color 0 0 0 0)
-	)
-	(junction
 		(at 63.5 49.53)
 		(diameter 0)
@@
 	)
 	(junction
+		(at 77.47 29.21)
+		(diameter 0)
+		(color 0 0 0 0)
+	)
+	(junction
 		(at 246.38 118.11)
 		(diameter 0)
@@
 	(wire
 		(pts
-			(xy 77.47 27.94) (xy 77.47 29.21)
-		)
-		(stroke
-			(width 0)
-			(type default)
-		)
-	)
-	(wire
-		(pts
 			(xy 25.4 111.76) (xy 27.94 111.76)
 		)
@@
 	(wire
 		(pts
+			(xy 73.66 29.21) (xy 77.47 29.21)
+		)
+		(stroke
+			(width 0)
+			(type default)
+		)
+	)
+	(wire
+		(pts
 			(xy 25.4 81.28) (xy 27.94 81.28)
 		)
@@
 	(wire
 		(pts
-			(xy 63.5 29.21) (xy 77.47 29.21)
+			(xy 63.5 29.21) (xy 66.04 29.21)
 		)
 		(stroke
@@
 	(wire
 		(pts
+			(xy 77.47 29.21) (xy 77.47 27.94)
+		)
+		(stroke
+			(width 0)
+			(type default)
+		)
+	)
+	(wire
+		(pts
 			(xy 127 58.42) (xy 127 59.69)
 		)
@@
 					(unit 1)
 				)
+			)
+		)
+	)
+	(symbol
+		(lib_id "Diode:PMEG2010BER")
+		(at 69.85 29.21 180)
+		(unit 1)
+		(body_style 1)
+		(exclude_from_sim no)
+		(in_bom yes)
+		(on_board yes)
+		(in_pos_files yes)
+		(dnp no)
+		(fields_autoplaced yes)
+		(property "Reference" "D1"
+			(at 70.1675 22.86 0)
+			(show_name no)
+			(do_not_autoplace no)
+			(effects
+				(font
+					(size 1.27 1.27)
+				)
+			)
+		)
+		(property "Value" "PMEG2010BER"
+			(at 70.1675 25.4 0)
+			(show_name no)
+			(do_not_autoplace no)
+			(effects
+				(font
+					(size 1.27 1.27)
+				)
+			)
+		)
+		(property "Footprint" "Diode_SMD:Nexperia_CFP3_SOD-123W"
+			(at 69.85 24.765 0)
+			(hide yes)
+			(show_name no)
+			(do_not_autoplace no)
+			(effects
+				(font
+					(size 1.27 1.27)
+				)
+			)
+		)
+		(property "Datasheet" "https://assets.nexperia.com/documents/data-sheet/PMEG2010BER.pdf"
+			(at 69.85 29.21 0)
+			(hide yes)
+			(show_name no)
+			(do_not_autoplace no)
+			(effects
+				(font
+					(size 1.27 1.27)
+				)
+			)
+		)
+		(property "Description" "20V, 1A low Vf MEGA Schottky barrier rectifier, SOD-123W"
+			(at 69.85 29.21 0)
+			(hide yes)
+			(show_name no)
+			(do_not_autoplace no)
+			(effects
+				(font
+					(size 1.27 1.27)
+				)
+			)
+		)
+		(pin "2"
+		)
+		(pin "1"
+		)
+		(instances
+			(project "memboard"
+				(path "/e4fac793-4acb-4ee2-a590-427dced759a1"
+					(reference "D1")
+					(unit 1)
+				)
